File: Design/Thermostat.sch (KiCad schematic (older format))
At the start: 31 parts, among them J1 BARREL_JACK, J2 CONN_01X01_MALE, J3 CONN_01X01_MALE, J4 CONN_01X01_MALE, J5 CONN_01X01_MALE, J6 CONN_01X01_MALE, J7 CONN_01X01_MALE, J8 Screw_Terminal_1x03, Q1 BC547, SW1 SW_Push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

Commit message: Add a recommendation to enabling the BOD
Other:
- note added: "Fuses ("0" means programmed):\n1. CKSEL3:0 = 0100 (enabling the Internal Calibrated RC Oscillator @ 8 MHz);\n2. BODEN = 0, BODLEVEL = 0, SUT1:0 = 00 (enabling the Internal Brown-out Detector).\n\nNotes:\n1. D2 is a green LED (heating is disabled), D3 is a red LED (heating is enabled)."
- note removed: "Notes:\n1. CKSEL3:0 = 0100 (internal calibrated RC oscillator @ 8 MHz);\n2. D2 is a green LED (heating is disabled), D3 is a red LED (heating is enabled)."
Changed lines of the file:
@@
 Sheet 1 1
 Title "Thermostat on ATmega8A, DS18B20 and 7-segment Display"
-Date "2017-07-30"
-Rev "3.0"
+Date "2017-10-07"
+Rev "3.1"
 Comp "Artyom Protaskin"
 Comment1 ""
@@
 	6200 4600 6200 5300
 Text Notes 550  7700 0    60   ~ 0
-Notes:\n1. CKSEL3:0 = 0100 (internal calibrated RC oscillator @ 8 MHz);\n2. D2 is a green LED (heating is disabled), D3 is a red LED (heating is enabled).
+Fuses ("0" means programmed):\n1. CKSEL3:0 = 0100 (enabling the Internal Calibrated RC Oscillator @ 8 MHz);\n2. BODEN = 0, BODLEVEL = 0, SUT1:0 = 00 (enabling the Internal Brown-out Detector).\n\nNotes:\n1. D2 is a green LED (heating is disabled), D3 is a red LED (heating is enabled).
 $EndSCHEMATC
